File: GateController.sch (KiCad schematic (older format))
At the start: 8 parts, among them P1 Power, P2 Analog, P3 Digital, P4 Digital, P5 CONN_01X01, P6 CONN_01X01, P7 CONN_01X01, P8 CONN_01X01

Commit message: Bring AM work in
Parts:
- added C1: C_Small, symbol Device:C_Small
- added D1, D2, D3: DIODE, symbol AM2:DIODE-Microtan_65_CPU-cache
- added D4: DIODE, symbol pspice:DIODE
- added K1, K2: RAYEX-L90, Relay_THT:Relay_SPDT_RAYEX-L90, symbol Relay:RAYEX-L90
- added M1, M2: N-CHANNEL-MOSFET-BSS138, SOT23-3, symbol AM1:GeekAmmo_N-CHANNEL-MOSFET-BSS138
- added M3: Motor_DC, symbol Motor:Motor_DC
- added R1: R_Small, symbol Device:R_Small
Connections:
- net +5V: now also D3.2 (K)
- net 1(Tx): now also M1.1 (G)
- net 2: now also M2.1 (G)
- net 5(**): now also C1.1, D3.1 (A), D4.2 (A), R1.1
- net GND: now also C1.2, D4.1 (K), K1.14, K2.14, M1.2 (S), M2.2 (S)
- new net: K1.11A, K1.11B, M3.2 (-)
- new net: D1.1 (A), K1.A1, M2.3 (D)
- new net: K2.11A, K2.11B, M3.1 (+)
- new net: D2.1 (A), K2.A2, M1.3 (D)
- new net +24V: D1.2 (K), D2.2 (K), K1.12, K1.A2, K2.12, K2.A1
- new net MAGICEYE: R1.2
- no-connect marks 5 -> 23
Other:
- note added: "INPUT"
- note added: "MOTOR\nCONTROL"
